File: Netzteil_Darlington_v2.sch (EAGLE design)
At the start: 155 parts, among them IC10 LT4320DIL08, IC11 OPA2197, IC13 OPA2197, IC15 LD33V, IC17 7815TV, IC2 OPA2197, IC4 VXO78012-1000, IC5 LD33V, IC6 VXO7805-1000, IC7 MCP4922, IC8 LTC6102HMS8#PBF, IC9 LM334, T1 IRLL110TRPBF, T10 BC847ALT1G, T11 BC847ALT1G, T12 DMG2302UK-7, T13 DMG2302UK-7, T14 DMG2302UK-7, T2 BC847ALT1G, T3 BD139, T4 2N5401, T5 TIP3055, T6 TIP3055, T7 BD139, T8 BC847ALT1G

Commit message: update to latest version
Parts:
- removed C44: 10µ / C3216X7R1E106M160AB, goujine:CC/1206
- removed C46: 100n, goujine:CC/0805
- removed CRNT_READ: (no value), jumper:JP2E
- removed D11: EDZV13B, neumluc:ZD
- removed D13: 1N4007, diode:DIODE-DO214AA
- removed R25: 347k 1%, neumluc:R-SMD0805
- removed R46: 10k, neumluc:R-SMD0805
- removed T8: BC847ALT1G, neumluc:T-NPNSOT23-BEC
- added C10, C17: 100n/16V, goujine:C
- added C14, C18, C41: 1µ/16V, goujine:CC/0805
- added C21: 330n, goujine:CC/0805
- added C28: 100n, goujine:CC/0805
- added C32, C37: 1µ/50V, goujine:CC/0805
- added C34: 10µ/16V, goujine:CC/0805
- added C40: 100n/50V, goujine:CC/0805
- added IC1: NCP718BSN330T1G, neumluc:NCP718
- added IC12: REF5040, neumluc:REF50XXVSSOP8
- added IC18, IC19: ADS1015, SparkFun-IC-Conversion:ADS1015
- added L6, L8: MPZ2012S601AT000, neumluc:L0805
- added R13: 10k, neumluc:R-SMD0603
- added R17: 2k2, neumluc:R-SMD0805
- added R19: 1.27R, neumluc:R-SMD0805
- C22, C29: device goujine:CC/0805 -> goujine:C
- C35: value 100n -> 1µ/50V
- C36: value 100n -> 1µ/16V
- C45: value 10µ / C3216X7R1E106M160AB -> 1µ/16V; device goujine:CC/1206 -> goujine:CC/0805
- C7: value 470n -> 100n/16V; device goujine:CC/0805 -> goujine:C
- C8: value 100n -> 10µ/16V
- C9: value 10µ / C3216X7R1E106M160AB -> 100n/16V; device goujine:CC/1206 -> goujine:C
- D4: value MMSD4148T1G opt -> 1N4007; device adafruit:DIODESOD-123 -> diode:DIODE-DO214AA
- IC17: value 7815TV -> 7818TV; device linear:7815TV -> linear:7818TV
- IC3: value (none) -> DAC8311; device neumluc:REF3120 -> neumluc:DAC8X11
- IC5: value LD33V -> 7815TV; device neumluc:LD33V -> linear:7815TV
- IC7: value MCP4922 -> DAC8311; device neumluc:MCP4922 -> neumluc:DAC8X11
- IC9: value LM334 -> NCP718BSN330T1G; device neumluc:LM334 -> neumluc:NCP718
- R1: value 1M -> 2k2 5%; device neumluc:R-SMD0603 -> neumluc:R-SMD0805
- R12: value 10R 1% -> 10k; device neumluc:R-SMD0805 -> neumluc:R-SMD0603
- R2: value 2.4k 0.1% PCF0805-13-2K4BT1 -> 10k 0.1% 10ppm
- R3: value 12k 0.1% ERA-6ARW123V -> 30k 0.1% 10ppm
- R4, R6: value 220R -> 10k; device neumluc:R-SMD0805 -> neumluc:R-SMD0603
- R42: value 681k 1% -> 390k 1%; device neumluc:R-SMD0603 -> neumluc:R-SMD0805
- T4: value 2N5401 -> DMMT5551-7-F; device neumluc:T-PNPTO92-G-EBC -> neumluc:T-NPN-DUAL
Connections:
- removed net AREF2048: C9.1, IC3.OUT, IC7.VREFA, IC7.VREFB, U$33.AREF
- removed net CRNT_READ_OP: CRNT_READ.2, IC13B.+IN
- removed net DAC_CS: IC7.CS, U$33.14/A0
- removed net DAC_SHDN: IC7.SHDN, U$33.A22/DAC1
- removed net MISO: U$33.12/MISO
- removed net N$39: C44.2, D13.A, IC5.VO, L5.1
- new net +27V: C1.+, C12.2, C19.2, C2.+, C21.1, C27.1, C42.1, C53.1, D4.C, D9.C, IC10.OUTP, IC17.VI, IC4.VI, IC5.VI, IC6.VI, IC8.V+, R5.I2, T15.D, T16.D
- new net +3.3V_A2: C14.2, IC9.OUT, L6.2
- new net +3.3V_LP: R4.2, R6.1, U$33.3V3_LO
- new net IDAC_CS: IC7.SYNC, U$33.15/A1
- new net N$18: IC19.ALERT/RDY, R12.2
- new net N$24: C17.1, IC18.ADDR, IC18.VDD, L8.1, R13.1
- new net N$25: C37.2, C40.2, IC12.VIN, L5.1
- new net N$32: C45.1, R19.2
- new net SCL: IC18.SCL, IC19.SCL, R4.1, U$33.19/A5/SCL
- new net SDA: IC18.SDA, IC19.SDA, R6.2, U$33.18/A4/SDA
- new net VDAC_CS: IC3.SYNC, U$33.14/A0
- new net VREF4096: C34.1, C41.1, C7.1, C8.1, C9.1, IC12.VOUT, IC3.AVDD/VREF, IC7.AVDD/VREF, R19.1
- net +15V: now also C28.1, C32.2, C35.2, D4.A, IC1.EN, IC1.IN, IC5.VO, IC9.EN, IC9.IN, L5.2, R1.1, R17.1; no longer C22.1, C29.1, C35.1, C43.1, D13.C, D9.A, IC13PWR.V+, IC17.VO, IC2PWR.V+, IC5.VI, R18.1, R46.1, T11.C
- net +18V: now also C22.1, C29.1, C43.1, D9.A, IC13PWR.V+, IC17.VO, IC2PWR.V+, R18.1, T11.C; no longer C1.+, C12.2, C19.2, C2.+, C27.1, C42.1, C53.1, D9.C, IC10.OUTP, IC17.VI, IC4.VI, IC6.VI, IC8.V+, R5.I2, T15.D, T16.D
- net +3.3V_A: now also C18.2, IC1.OUT, L8.2; no longer C36.2, C45.1, C46.1, C7.1, C8.1, IC3.IN, IC7.VDD, L5.2
- net +V_ADJ: now also T4.C2; no longer IC9.V+, T8.C
- net ADC_CH0: now also IC18.AIN2; no longer U$33.20/A6
- net ADC_CH1: now also IC19.AIN0; no longer U$33.33/A14
- net ADC_CH2: now also IC19.AIN2; no longer U$33.34/A15
- net ADC_CH3: now also IC18.AIN0; no longer U$33.19/A5/SCL
- net AGND: now also C10.2, C14.1, C17.2, C18.1, C21.2, C28.2, C32.1, C34.2, C35.1, C36.2, C37.1, C40.1, C41.2, IC1.GND, IC12.VSS, IC18.AIN1, IC18.AIN3, IC18.VSS, IC19.ADDR, IC19.AIN1, IC19.AIN3, IC19.VSS, IC7.VSS, IC9.GND, R17.2, SENSE.1, T4.E1, T4.E2; no longer C35.2, C36.1, C44.1, C46.2, D11.A, IC7.AVSS, IC7.LDAC, IC9.V-, R1.1, R12.2, T8.E
- net BTN_I_DOWN: now also U$33.37/A18; no longer U$33.39/A20
- net BTN_I_UP: now also U$33.36/A17; no longer U$33.38/A19
- net BTN_V_DOWN: now also U$33.35/A16; no longer U$33.37/A18
- net BTN_V_UP: now also U$33.34/A15; no longer U$33.36/A17
- net CRNT_READ: now also IC13B.+IN; no longer CRNT_READ.3
- net CRNT_READ_RAW: no longer CRNT_READ.1
- net ISET: now also IC7.VOUT; no longer IC7.VOUTA
- net MOSI: now also IC3.DIN, IC7.DIN; no longer IC7.SDI
- net N$10: no longer D4.C
- net N$11: now also R1.2, T4.B1, T4.B2, T4.C1; no longer R25.1, T8.B
- net N$14: now also C36.1, IC12.TRIM/NR; no longer D11.C, R25.2, R46.2
- net N$15: no longer R4.2
- net N$16: now also IC18.ALERT/RDY, R13.2; no longer IC9.R, R12.1
- net N$19: now also C10.1, IC19.VDD, L6.1, R12.1; no longer R1.2, T4.B
- net N$21: no longer T4.E
- net N$22: no longer D4.A, T4.C
- net N$4: no longer R6.1
- net N$5: no longer R6.2
- net N$8: no longer R4.1
- net SCK: now also IC3.SCLK, IC7.SCLK; no longer IC7.SCK
- net TH0: now also U$33.33/A14; no longer U$33.35/A16
- net VSET: now also IC3.VOUT; no longer IC7.VOUTB
Other:
- note added: "6,5mA Pulldown"
- moved on the sheet: C35, C36, D8, R1, R12, R31, R48, REL1, T1

Commit message: update to latest version
Parts:
- removed BTNS: (no value), con-lstb:MA05-1
- added I: (no value), con-lstb:MA03-1
- added SENSE_GND, V: (no value), jumper:JP1E
Connections:
- new net SENSE_GND: IC19.AIN1, SENSE_GND.1, SENSE_GND.2
- net +V_ADJ: now also REL12.S; no longer REL12.P
- net AGND: now also I.3, REL13.S; no longer BTNS.5, IC19.AIN1, REL13.P, SENSE.1
- net BTN_I_DOWN: now also I.2, U$33.17/A3; no longer BTNS.4, U$33.37/A18
- net BTN_I_UP: now also I.1, U$33.16/A2; no longer BTNS.3, U$33.36/A17
- net BTN_V_DOWN: now also V.2; no longer BTNS.2
- net BTN_V_UP: now also V.1; no longer BTNS.1
- net GND_OUT_CON: now also REL13.P; no longer REL13.S
- net SENSE: now also SENSE.1
- net V_OUT_CON: now also REL12.P; no longer REL12.S

Commit message: Update to v1.9
Parts:
- removed C29: 100n, goujine:C
- removed C50: 10n, goujine:CC/0805
- removed D12: 1N4007, diode:DIODE-DO214AA
- removed DSPLY2, LED, SENSE, SENSE_GND, V: (no value), jumper:JP1E
- removed DSPLY_LED: (no value), neumluc:MA03-1
- removed ESP: (no value), con-lstb:MA06-1
- removed I: (no value), con-lstb:MA03-1
- removed IC11, IC13: OPA2197, goujine:DUAL-OPVSOP8
- removed R15: 10.1k 0.1% RN732ATTD1012B25, neumluc:R-SMD0805
- removed R31: 360R, neumluc:R-SMD0805
- removed R38: 4.7k, neumluc:R-SMD0805
- removed R39: 100R, neumluc:R-SMD0805
- removed T10: BC847ALT1G, neumluc:T-NPNSOT23-BEC
- added BTN, SV1, SV2: (no value), neumluc:JST-PH-2.0-2P
- added C33, C44: 100µ/50V, goujine:C+3.5/8
- added ESP/BTNS: (no value), neumluc:JST-PH-2.0-8P
- added IC14: QUAD-OPVOPA4197, neumluc:QUAD-OPVOPA4197
- added R25, R26: 1k 1% 1/8W, neumluc:R-SMD0805
- added SINK: (no value), jumper:JP1E
- added SV5: (no value), neumluc:JST-PH-2.0-5P
- AC1: OC_MOUSER (none) -> 710-691311500002; OC_MOUSER_ADD (none) -> 693-8601.2001.08; OC_MOUSER_ADD2 (none) -> 693-3101.0010
- AC2: OC_MOUSER (none) -> 710-691311500002; OC_MOUSER_ADD (none) -> 693-8601.2001.08
- C1, C2: value UVZ1H103MRD -> 10000µ/50V; OC_MOUSER (none) -> 647-UVZ1H103MRD
- C10, C17, C7, C9: device goujine:C -> goujine:CC/0805; OC_MOUSER (none) -> 810-C2012X7R2A104K
- C11: value 330n opt -> 330n opt/50V; OC_MOUSER (none) -> 80-C0805C334K5RECTU
- C12, C19: OC_MOUSER (none) -> 81-GRM32ER71H106MA2L
- C13: value 100n opt -> 100n opt/50V; OC_MOUSER (none) -> 810-C2012X7R2A104K
- C14, C18, C36, C41, C45: OC_MOUSER (none) -> 963-UMK212B7105KG-T
- C15: value 100µ/50V EEU-FR1H101 -> 100µ/50V; OC_MOUSER (none) -> 667-EEU-FR1H101
- C16: value 10µ/16V -> 10µ/25V; device we-rcl:CAPACITOR-1210 -> goujine:CC/1206; OC_MOUSER (none) -> 963-TMK316AB7106KL-T
- C20: device we-rcl:CAPACITOR-1210 -> goujine:CC/1206; OC_MOUSER (none) -> 963-TMK316AB7106KL-T
- C21, C42: value 330n -> 330n/50V; OC_MOUSER (none) -> 80-C0805C334K5RECTU
- C22: value 100n -> 100n/35V; device goujine:C -> goujine:CC/0805; OC_MOUSER (none) -> 810-C2012X7R2A104K
- C23, C30, C39, C49: value 10µ / C3216X7R1E106M160AB -> 10µ/16V; OC_MOUSER (none) -> 963-TMK316AB7106KL-T
- C24, C3, C31, C38, C48: value 100n -> 100n/16V; OC_MOUSER (none) -> 810-C2012X7R2A104K
- C25, C28, C43: value 100n -> 100n/35V; OC_MOUSER (none) -> 810-C2012X7R2A104K
- C26: value 100n -> 1n/50V; OC_MOUSER (none) -> 603-CC805KRX7R0BB102
- C27: value 100n -> 100n/50V; OC_MOUSER (none) -> 810-C2012X7R2A104K
- C32, C35, C37: value 1µ/50V -> 1µ/35V; OC_MOUSER (none) -> 963-UMK212B7105KG-T
- C34, C8: device goujine:CC/0805 -> goujine:CC/1206; OC_MOUSER (none) -> 963-TMK316AB7106KL-T
- C4: value 10n -> 10n/50V; OC_MOUSER (none) -> 80-C0805C103K1R
- C40: value 100n/50V -> 100n/35V; OC_MOUSER (none) -> 810-C2012X7R2A104K
- C47, C51: value 10n -> 10n/16V; OC_MOUSER (none) -> 80-C0805C103K1R
- C5: value 1n -> 1n/50V; OC_MOUSER (none) -> 603-CC805KRX7R0BB102
- C52: value 22p opt -> 22p opt/35V C0G; OC_MOUSER (none) -> 603-CC805JRNPO9BN220
- C53: value (none) -> 1µ/50V; OC_MOUSER (none) -> 603-CC126KKX7R9BB105
- C6: value 22pF -> 22pF/35V C0G; OC_MOUSER (none) -> 603-CC805JRNPO9BN220
- D1, D2, D3: OC_MOUSER (none) -> 511-BAT54FILMY
- D14, D6: value CDBA5200-HF -> CGRB307-G; device neumluc:CDBA5200-HF -> neumluc:DWIDE; OC_MOUSER (none) -> 750-CGRB307-G
- D4, D8, D9: value 1N4007 -> CGRB307-G; device diode:DIODE-DO214AA -> neumluc:DWIDE; OC_MOUSER (none) -> 750-CGRB307-G
- DSPLY: device con-lstb:MA07-1 -> neumluc:JST-PH-2.0-7P
- ENC: device con-lstb:MA03-1 -> neumluc:JST-PH-2.0-3P
- FAN: device con-lstb:MA04-1 -> neumluc:JST-PH-2.0-4P
- GND_OUT_CON: OC_MOUSER (none) -> 710-691311500002
- HS2: OC_MOUSER (none) -> 567-OMNI-UNI-41-75; OC_MOUSER_ADD (none) -> 567-OMNI-UC; OC_MOUSER_ADD2 (none) -> 567-CD-02-05-247
- IC1, IC9: OC_MOUSER (none) -> 863-NCP718BSN330T1G
- IC10: OC_MOUSER (none) -> 584-LT4320HN8-1#PBF
- IC12: OC_MOUSER (none) -> 595-REF5040AIDGKR
- IC15: OC_MOUSER (none) -> 511-LD1117V33
- IC17: OC_MOUSER (none) -> 511-L7818CV-DG
- IC18, IC19: value ADS1015 -> ADS1115; device SparkFun-IC-Conversion:ADS1015 -> neumluc:ADS1015; OC_MOUSER (none) -> 595-ADS1115IDGSR
- IC2: value OPA2197 -> (none)
- IC3, IC7: OC_MOUSER (none) -> 595-DAC8311IDCKR
- IC4: OC_MOUSER (none) -> 490-VXO7812-1000
- IC5: OC_MOUSER (none) -> 511-L7815CV-DG
- IC6: OC_MOUSER (none) -> 490-VXO7805-1000
- IC8: OC_MOUSER (none) -> 584-LTC6102HMS8#PBF
- L1, L2, L3, L4, L5, L6, L8: OC_MOUSER (none) -> 810-MPZ2012S601AT000
- R1: value 2k2 5% -> 12k 0.5% 50 ppm 1/10W; OC_MOUSER (none) -> 754-RR1220P-123D
- R10: value 4.7k opt -> 4.7k opt 1% 1/10W; OC_MOUSER (none) -> 652-CR0805FX-4701ELF
- R11, R16: value 22R -> 22R 5% 1/10W; OC_MOUSER (none) -> 652-CR0805JW-220ELF
- R12: value 10k -> 221R 0.5% 50ppm 1/10W; device neumluc:R-SMD0603 -> neumluc:R-SMD0805; OC_MOUSER (none) -> 754-RR1220P-2210D-M
- R13: value 10k -> 1k 0.5% 50 ppm 1/10W; device neumluc:R-SMD0603 -> neumluc:R-SMD0805; OC_MOUSER (none) -> 754-RR1220P-102D
- R14: value 90.9k 0.1% RN73C2A90K9BTDF -> 10R 0.5% 50 ppm 1/4W; OC_MOUSER (none) -> 660-SG73G2ATTD10R0D
- R17: value 2k2 -> 2k2 5% 1/8W; OC_MOUSER (none) -> 652-CR0805JW-222ELF
- R18: value 2k2 -> 1k 1% 1/8W; OC_MOUSER (none) -> 652-CR0805FX-1001ELF
- R19: value 1.27R -> 1.27R 1% 1/10W; OC_MOUSER (none) -> 71-CRCW08051R27FKEA
- R2: OC_MOUSER (none) -> 667-ERA-6ARW103V
- R20, R21: value 0R1 0.5% -> 0R1 0.5% 7W; OC_MOUSER (none) -> 66-SLN5TTED82L0D
- R22, R32: value 10.1k 0.1% RN732ATTD1012B25 -> 10.1k 0.1% 10ppm 1/10W; OC_MOUSER (none) -> 660-RN732ATTD1012B25
- R23, R30: value 90.9k 0.1% RN73C2A90K9BTDF -> 90.9k 0.1% 10ppm 1/10W; OC_MOUSER (none) -> 279-RN73CA-90.9K
- R24: value 1k opt -> 1k 1% 1/10W; OC_MOUSER (none) -> 652-CR0805FX-1001ELF
- R28, R29: value 220R -> 220R 5% 1/10W; OC_MOUSER (none) -> 652-CR0805FX-2200ELF
- R3: OC_MOUSER (none) -> 667-ERA-6ARW303V
- R35, R40: value 4.7k -> 4.7k 5% 1/10W; OC_MOUSER (none) -> 652-CR0805FX-4701ELF
- R36: OC_MOUSER (none) -> 594-NTCLE213E3104HXB
- R37: value 100R -> 2.2k 5% 1/8W; OC_MOUSER (none) -> 652-CR0805JW-101ELF
- R4, R6: value 10k -> 10k 5% 1/10W; device neumluc:R-SMD0603 -> neumluc:R-SMD0805; OC_MOUSER (none) -> 652-CR0805-JW-103ELF
- R41: value 100R -> 100R 5% 1/10W; OC_MOUSER (none) -> 652-CR0805JW-101ELF
- R42: value 390k 1% -> 65k 1% 1/10W; OC_MOUSER (none) -> 652-CR0805FX-3903ELF
- R43: value 5k 0.1% low ppm TNPW12065K00BEEN -> 5k 0.1% 25ppm; OC_MOUSER (none) -> 71-TNPW12065K00BEEN
- R44, R45: value 100R 0.1% low ppm PCF0805-13-100RBT1 -> 100R 0.1% 5ppm 1/10W; OC_MOUSER (none) -> 756-PCF080513100RBT1
- R48, R7: value 10k -> 10k 5% 1/10W; OC_MOUSER (none) -> 652-CR0805-JW-103ELF
- R5: value 10m -> 10m 0.1% 15ppm 0.5W; OC_MOUSER (none) -> 71-CSM25120R0100BST
- R8: value 47k -> 47k 1% 1/10W; OC_MOUSER (none) -> 652-CR0805FX-4702ELF
- R9: value 4.7k -> 4.7k 1% 1/10W; OC_MOUSER (none) -> 652-CR0805FX-4701ELF
- REL1: OC_MOUSER (none) -> 653-G2R-2-DC12
- SG1: OC_MOUSER (none) -> 254-EMB73-RO
- T1: value IRLL110TRPBF -> PMV130ENEAR; device goujine:T-NMOSFDT457N -> neumluc:T-NMOSIRLML2502PBF; OC_MOUSER (none) -> 771-PMV130ENEAR
- T11, T2: OC_MOUSER (none) -> 863-BC847ALT1G
- T12, T13, T14: value DMG2302UK-7 -> PMV130ENEAR; OC_MOUSER (none) -> 771-PMV130ENEAR
- T15, T16, T17, T18: value (none) -> IRFR7546TRPBF; OC_MOUSER (none) -> 942-IRFR7546TRPBF
- T3, T7: OC_MOUSER (none) -> 511-BD139-10
- T4: value DMMT5551-7-F -> PMV130ENEAR; device neumluc:T-NPN-DUAL -> neumluc:T-NMOSIRLML2502PBF; OC_MOUSER (none) -> 771-PMV130ENEAR
- T5, T6: OC_MOUSER (none) -> 863-TIP3055G
- U$33: OC_MOUSER (none) -> 474-DEV-14055
- VOUT: OC_MOUSER (none) -> 710-691311500002; OC_MOUSER_ADD (none) -> 565-72912-2; OC_MOUSER_ADD2 (none) -> 565-6883
Connections:
- removed net ADC_CH1: C50.1, IC19.AIN0, R39.2
- removed net ADC_SENSE: C25.1, IC11A.+IN, R14.1, R15.2
- removed net N$37: R31.1, R48.2, T1.G
- removed net N$40: IC11B.OUT, T2.B
- removed net N$42: IC11A.OUT, T10.B
- removed net N$43: IC11A.-IN, R38.1, R39.1, T10.E
- removed net N$44: IC13B.OUT, T11.B
- removed net SENSE: R14.2, SENSE.1, SENSE.2
- removed net SENSE_GND: IC19.AIN1, SENSE_GND.1, SENSE_GND.2
- new net 3.3V_A2_FILTERED: C10.1, IC19.VDD, L6.1, R1.1, SV1.2
- new net 3.3V_TH: R42.1, SV2.2
- new net N$26: R18.2, R25.1
- new net N$30: R25.2, R26.1
- new net N$31: C6.1, IC14C.-IN, R2.2, R3.2, R8.2
- new net N$33: C26.1, IC2A.OUT, T4.G
- new net N$34: SINK.2, T4.D
- new net TH0_ADC: IC19.AIN0, SV1.1
- net +15V: now also C25.1, IC2PWR.V+; no longer C26.1, IC11PWR.V+, R1.1, R42.1, T10.C
- net +18V: now also IC14PWR.V+; no longer C29.1, IC13PWR.V+, IC2PWR.V+
- net +27V: now also C33.+, C44.+
- net +3.3V: now also DSPLY.6, ESP/BTNS.4; no longer DSPLY.2, DSPLY2.2, ESP.4
- net +5V_INT_D: no longer D12.C
- net +V_ADJ: now also SINK.1; no longer T4.C2
- net ADC_CH0: now also IC18.AIN0; no longer IC18.AIN2
- net ADC_CH3: now also IC18.AIN2; no longer IC18.AIN0
- net ADC_VOUT: now also IC2B.+IN; no longer IC11B.+IN
- net AGND: now also IC14PWR.V-, R12.2, R14.2, R26.2, U$33.GND2; no longer C26.2, C29.2, C50.2, I.3, IC11PWR.V-, IC13PWR.V-, R15.1, R18.2, R38.2, T4.E1, T4.E2
- net BTN_I_DOWN: now also BTN.2; no longer I.2
- net BTN_I_UP: now also BTN.1; no longer I.1
- net BTN_V_DOWN: now also ESP/BTNS.8, U$33.33/A14; no longer U$33.35/A16, V.2
- net BTN_V_UP: now also ESP/BTNS.7; no longer V.1
- net CRNT_READ: now also IC14B.+IN, IC14D.-IN; no longer IC13B.+IN, IC2B.-IN
- net DSPLY_CS: now also DSPLY.1; no longer DSPLY.7
- net DSPLY_DC: now also DSPLY.5; no longer DSPLY.3
- net DSPLY_RST: now also DSPLY.2; no longer DSPLY.6
- net ESP-IO: now also ESP/BTNS.5, U$33.35/A16; no longer ESP.5, U$33.10/CS
- net ESP-RST: now also ESP/BTNS.3; no longer ESP.3
- net ESP-RX: now also ESP/BTNS.2, U$33.32/A13; no longer ESP.2, U$33.31/A12
- net ESP-TX: now also ESP/BTNS.1, U$33.31/A12; no longer ESP.1, U$33.32/A13
- net ISET: now also IC14D.+IN; no longer IC2B.+IN
- net MOSI: now also DSPLY.3; no longer DSPLY.5
- net N$11: now also IC2A.+IN, R12.1; no longer T4.B1, T4.B2, T4.C1
- net N$16: now also R14.1, T4.S; no longer IC18.ALERT/RDY
- net N$18: now also C26.2, IC2A.-IN, R13.1; no longer IC19.ALERT/RDY, R12.2
- net N$19: now also IC2B.OUT, T2.B; no longer C10.1, IC19.VDD, L6.1, R12.1
- net N$20: now also SV5.1; no longer LED.1
- net N$21: now also IC14C.OUT; no longer IC2A.OUT
- net N$23: now also SV5.2; no longer LED.2
- net N$24: no longer R13.1
- net N$35: no longer D12.A
- net N$41: now also IC2B.-IN; no longer IC11B.-IN
- net N$45: now also IC14B.-IN; no longer IC13B.-IN
- net N$46: now also SV5.4; no longer DSPLY_LED.2
- net N$48: now also SV5.5; no longer DSPLY_LED.3
- net N$6: now also IC14B.OUT, T11.B; no longer C6.1, IC2A.-IN, R2.2, R3.2, R8.2
- net N$7: now also SV5.3; no longer DSPLY_LED.1
- net OVRCRNT_DET: now also IC14A.+IN, IC14D.OUT; no longer IC13A.+IN, IC2B.OUT
- net OVRCRNT_DET_BUF: now also IC14A.-IN, IC14A.OUT; no longer IC13A.-IN, IC13A.OUT
- net REL-OUT: now also R48.2, T1.G; no longer R31.2
- net TH0: now also SV2.1; no longer U$33.33/A14
- net VSET: now also IC14C.+IN; no longer IC2A.+IN
- net VSS: now also C33.-, C44.-, DSPLY.7, ESP/BTNS.6; no longer DSPLY.1, DSPLY2.1, ESP.6
Other:
- note removed: "6,5mA Pulldown"
- moved on the sheet: C14, C25, C26, IC2A, IC2B, L6, R1, R12, R13, R14, R18, R28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
